File: chip.sch (KiCad schematic (older format))
At the start: 43 parts, among them J1 Conn_01x04, J2 Conn_01x07_Male, J3 USB_C_Receptacle_USB2.0, J4 Conn_01x02, Q1 UMH3N, SW1 SW_SPST, SW2 SW_SPST, U1 ESP32-WROOM-32D, U2 MT3420C, U3 CP2104

Commit message: last changes before moving to 5.99
Parts:
- added C?: 100n, Capacitor_SMD:C_0603_1608Metric, symbol Device:C
- added R19: 100R, Resistor_SMD:R_0603_1608Metric, symbol Device:R
- added U?: SN74LV1T125, symbol SN74LV1T125:SN74LV1T125
Connections:
- wire segments 131 -> 139
Other:
- note added: "0,6V"
- note added: "3,3V"
- moved on the sheet: BZ1
Changed lines of the file:
@@
 Connection ~ 3500 900
 Wire Wire Line
-	3950 1900 7300 1900
-Wire Wire Line
-	7300 1900 7300 1350
-Wire Wire Line
-	7300 1350 8500 1350
+	3950 1900 6350 1900
 $Comp
 L Switch:SW_SPST SW2
@@
 L Device:Buzzer BZ1
 U 1 1 60E4F1A7
-P 6500 2200
-F 0 "BZ1" H 6652 2229 50  0000 L CNN
-F 1 "Buzzer" H 6652 2138 50  0000 L CNN
-F 2 "Buzzer_Beeper:Buzzer_Murata_PKMCS0909E4000-R1" V 6475 2300 50  0001 C CNN
-F 3 "~" V 6475 2300 50  0001 C CNN
-F 4 "C391035" H 6500 2200 50  0001 C CNN "LCSC"
-	1    6500 2200
-	1    0    0    -1
-$EndComp
-Wire Wire Line
-	3950 2100 6400 2100
-Wire Wire Line
-	6400 2300 6400 2350
+P 5950 2200
+F 0 "BZ1" H 6102 2229 50  0000 L CNN
+F 1 "Buzzer" H 6102 2138 50  0000 L CNN
+F 2 "Buzzer_Beeper:Buzzer_Murata_PKMCS0909E4000-R1" V 5925 2300 50  0001 C CNN
+F 3 "~" V 5925 2300 50  0001 C CNN
+F 4 "C391035" H 5950 2200 50  0001 C CNN "LCSC"
+	1    5950 2200
+	1    0    0    -1
+$EndComp
+Wire Wire Line
+	3950 2100 5850 2100
+Wire Wire Line
+	5850 2300 5850 2350
 $Comp
 L power:GND #PWR05
 U 1 1 60E58EAF
-P 6400 2350
-F 0 "#PWR05" H 6400 2100 50  0001 C CNN
-F 1 "GND" H 6405 2177 50  0000 C CNN
-F 2 "" H 6400 2350 50  0001 C CNN
-F 3 "" H 6400 2350 50  0001 C CNN
-	1    6400 2350
+P 5850 2350
+F 0 "#PWR05" H 5850 2100 50  0001 C CNN
+F 1 "GND" H 5855 2177 50  0000 C CNN
+F 2 "" H 5850 2350 50  0001 C CNN
+F 3 "" H 5850 2350 50  0001 C CNN
+	1    5850 2350
 	1    0    0    -1
 $EndComp
@@
 Wire Wire Line
 	9750 4200 9850 4200
+Text Notes 9350 5800 0    50   ~ 0
+0,6V
+Text Notes 9350 5450 0    50   ~ 0
+3,3V
+$Comp
+L power:GND #PWR0163
+U 1 1 610811FE
+P 7050 1350
+F 0 "#PWR0163" H 7050 1100 50  0001 C CNN
+F 1 "GND" H 7055 1177 50  0000 C CNN
+F 2 "" H 7050 1350 50  0001 C CNN
+F 3 "" H 7050 1350 50  0001 C CNN
+	1    7050 1350
+	1    0    0    -1
+$EndComp
+$Comp
+L power:+5V #PWR0162
+U 1 1 60FE9C4F
+P 7850 750
+F 0 "#PWR0162" H 7850 600 50  0001 C CNN
+F 1 "+5V" H 7865 923 50  0000 C CNN
+F 2 "" H 7850 750 50  0001 C CNN
+F 3 "" H 7850 750 50  0001 C CNN
+	1    7850 750
+	1    0    0    -1
+$EndComp
+$Comp
+L Device:R R19
+U 1 1 610EBFC2
+P 6500 1900
+F 0 "R19" V 6293 1900 50  0000 C CNN
+F 1 "100R" V 6384 1900 50  0000 C CNN
+F 2 "Resistor_SMD:R_0603_1608Metric" V 6430 1900 50  0001 C CNN
+F 3 "~" H 6500 1900 50  0001 C CNN
+F 4 "C105588" H 6500 1900 50  0001 C CNN "LCSC"
+	1    6500 1900
+	0    1    1    0
+$EndComp
+Wire Wire Line
+	7700 1350 8500 1350
+$Comp
+L SN74LV1T125:SN74LV1T125 U?
+U 1 1 610D2FDD
+P 7400 1200
+F 0 "U?" H 7400 1615 50  0000 C CNN
+F 1 "SN74LV1T125" H 7400 1524 50  0000 C CNN
+F 2 "" H 7400 1500 50  0001 C CNN
+F 3 "" H 7400 1500 50  0001 C CNN
+	1    7400 1200
+	1    0    0    -1
+$EndComp
+$Comp
+L Device:C C?
+U 1 1 610E4E4B
+P 7850 950
+AR Path="/60CA433D/610E4E4B" Ref="C?"  Part="1"
+AR Path="/60D0FE54/610E4E4B" Ref="C?"  Part="1"
+F 0 "C?" H 7965 996 50  0000 L CNN
+F 1 "100n" H 7965 905 50  0000 L CNN
+F 2 "Capacitor_SMD:C_0603_1608Metric" H 7888 800 50  0001 C CNN
+F 3 "~" H 7850 950 50  0001 C CNN
+F 4 "C14663" H 7850 950 50  0001 C CNN "LCSC"
+	1    7850 950
+	1    0    0    -1
+$EndComp
+$Comp
+L power:GND #PWR?
+U 1 1 610E9BFC
+P 7850 1100
+F 0 "#PWR?" H 7850 850 50  0001 C CNN
+F 1 "GND" H 7855 927 50  0000 C CNN
+F 2 "" H 7850 1100 50  0001 C CNN
+F 3 "" H 7850 1100 50  0001 C CNN
+	1    7850 1100
+	1    0    0    -1
+$EndComp
+Wire Wire Line
+	7850 750  7850 800
+Wire Wire Line
+	7850 800  7700 800
+Wire Wire Line
+	7700 800  7700 1050
+Connection ~ 7850 800
+Wire Wire Line
+	7100 1200 6950 1200
+Wire Wire Line
+	6950 1200 6950 1900
+Wire Wire Line
+	6650 1900 6950 1900
+Wire Wire Line
+	7100 1050 7050 1050
+Wire Wire Line
+	7050 1050 7050 1350
+Wire Wire Line
+	7050 1350 7100 1350
+Connection ~ 7050 1350
 $EndSCHEMATC
